Commit message: Update URDF to match robot structure

File: description/camera.xacro (robot description, xacro)
@@ -4,12 +4,12 @@
         <parent link="chassis"/>
         <child link="camera_link"/>
-        <origin xyz="0.305 0.0 0.08" rpy="0.0 0.0 0.0"/>
+        <origin xyz="${chassis_length} 0.0 0.098" rpy="0.0 0.0 0.0"/>
     </joint>
     <link name="camera_link">
         <visual>
             <geometry>
-                <box size="0.010 0.03 0.03"/>
+                <box size="0.01 0.094 0.03"/>
             </geometry>
-            <material name="red"/>
+            <material name="black"/>
          </visual>
     </link>
@@ -21,5 +21,5 @@
     <link name="camera_link_optical"></link>
     <gazebo reference="camera_link">
-       <material>Gazebo/Red</material>
+       <material>Gazebo/Black</material>
        <sensor name="camera" type="camera">
             <pose> 0 0 0 0 0 0 </pose>

File: description/lidar.xacro (robot description, xacro)
@@ -1,27 +1,29 @@
 <?xml version="1.0"?>
 <robot xmlns:xacro="http://www.ros.org/wiki/xacro" >
+    <xacro:property name="lidar_length" value="0.041"/>
+    <xacro:property name="lidar_radius" value="0.038"/>
     <joint name="laser_joint" type="fixed">
         <parent link="chassis"/>
         <child link="laser_frame"/>
-        <origin xyz="0.1 0.0 0.175" rpy="0.0 0.0 0.0"/>
+        <origin xyz="${chassis_length/2} 0.0 ${chassis_height+lidar_length/2}" rpy="0.0 0.0 0.0"/>
     </joint>
     <link name="laser_frame">
         <visual>
             <geometry>
-               <cylinder radius="0.05" length="0.04"/>
+               <cylinder radius="${lidar_radius}" length="${lidar_length}"/>
             </geometry>
-            <material name="red"/>
+            <material name="black"/>
          </visual>
          <collision>
             <geometry>
-               <cylinder radius="0.05" length="0.04"/>
+               <cylinder radius="${lidar_radius}" length="${lidar_length}"/>
             </geometry>
          </collision>
-         <xacro:inertial_cylinder mass="0.1" length="0.04" radius="0.05">
+         <xacro:inertial_cylinder mass="0.1" length="${lidar_length}" radius="${lidar_radius}">
             <origin xyz="0.0 0.0 0.0" rpy="0.0 0.0 0.0"/>
          </xacro:inertial_cylinder>
     </link>
     <gazebo reference="laser_frame">
-        <material>Gazebo/Red</material>
+        <material>Gazebo/Black</material>
         <sensor name="laser" type="ray">
             <pose> 0 0 0 0 0 0 </pose>

File: description/robot.urdf.xacro (robot description, xacro)
@@ -6,3 +6,4 @@
    <xacro:include filename="lidar.xacro"/>
    <xacro:include filename="camera.xacro"/>
+   <xacro:include filename="face.xacro"/>
 </robot>

File: description/robot_core.xacro (robot description, xacro)
@@ -2,4 +2,20 @@
 <robot xmlns:xacro="http://www.ros.org/wiki/xacro" >
    <xacro:include filename="inertial_macros.xacro"/>
+   <!-- unit meter -->
+   <xacro:property name="chassis_length" value="0.262"/>
+   <xacro:property name="chassis_width" value="0.154"/>
+   <xacro:property name="chassis_height" value="0.128"/>
+   <xacro:property name="chassis_mass" value="1.0"/>
+   <xacro:property name="wheel_radius" value="0.040"/>
+   <xacro:property name="wheel_thickness" value="0.035"/>
+   <xacro:property name="wheel_mass" value="0.05"/>
+   <xacro:property name="wheel_offset_x" value="0.04"/>
+   <xacro:property name="wheel_offset_y" value="0.107"/>
+   <xacro:property name="wheel_offset_z" value="0.0315"/>
+   <xacro:property name="caster_wheel_radius" value="0.0079"/>
+   <xacro:property name="caster_wheel_mass" value="0.01"/>
+   <xacro:property name="caster_wheel_offset_x" value="0.207"/>
+   <xacro:property name="caster_wheel_offset_y" value="0.0485"/>
+   <xacro:property name="caster_wheel_offset_z" value="${wheel_offset_z + wheel_radius - caster_wheel_radius}"/>
    <material name="white">
       <color rgba="1 1 1 1"/>
@@ -24,32 +40,33 @@
       <parent link="base_link"/>
       <child link="chassis"/>
-      <origin xyz="-0.1 0 0"/>
+      <origin xyz="${-wheel_offset_x} 0 0"/>
    </joint>
    <link name="chassis">
       <visual>
-         <origin xyz="0.15 0 0.075"/>
+         <origin xyz="${chassis_length/2} 0 ${chassis_height/2}"/>
          <geometry>
-            <box size="0.3 0.3 0.15"/>
+            <box size="${chassis_length} ${chassis_width} ${chassis_height}"/>
          </geometry>
-         <material name="white"/>
+         <material name="orange"/>
       </visual>
       <collision>
-         <origin xyz="0.15 0 0.075"/>
+         <origin xyz="${chassis_length/2} 0 ${chassis_height/2}"/>
          <geometry>
-            <box size="0.3 0.3 0.15"/>
+            <box size="${chassis_length} ${chassis_width} ${chassis_height}"/>
          </geometry>
       </collision>
-      <xacro:inertial_box mass="0.5" x="0.3" y="0.3" z="0.15">
-         <origin xyz="0.15 0.0 0.075" rpy="0.0 0.0 0.0"/>
+      <xacro:inertial_box mass="0.5" x="${chassis_length}" y="${chassis_width}" z="${chassis_height}">
+         <origin xyz="${chassis_length/2} 0 ${chassis_height/2}" rpy="0 0 0"/>
       </xacro:inertial_box>
    </link>
    <gazebo reference="chassis">
-      <material>Gazebo/White</material>
+      <material>Gazebo/Orange</material>
    </gazebo>
    <!--LEFT WHEEL LINK-->
+   <!-- <joint name="left_wheel_joint" type="continuous"> -->
    <joint name="left_wheel_joint" type="continuous">
       <parent link="base_link"/>
       <child link="left_wheel"/>
-      <origin xyz="0.0 0.175 0.0" rpy="-${pi/2} 0.0 0.0"/>
+      <origin xyz="0 ${wheel_offset_y} ${-wheel_offset_z}" rpy="-${pi/2} 0 0" />
       <axis xyz="0.0 0.0 1"/>
    </joint>
@@ -57,5 +74,5 @@
       <visual>
          <geometry>
-            <cylinder radius="0.05" length="0.04"/>
+            <cylinder radius="${wheel_radius}" length="${wheel_thickness}"/>
          </geometry>
          <material name="blue"/>
@@ -63,9 +80,9 @@
       <collision>
          <geometry>
-            <cylinder radius="0.05" length="0.04"/>
+            <sphere radius="${wheel_radius}"/>
          </geometry>
       </collision>
-      <xacro:inertial_cylinder mass="0.1" length="0.04" radius="0.05">
-         <origin xyz="0.0 0.0 0.0" rpy="0.0 0.0 0.0"/>
+      <xacro:inertial_cylinder mass="${wheel_mass}" length="${wheel_thickness}" radius="${wheel_radius}">
+         <origin xyz="0 0 0" rpy="0 0 0"/>
       </xacro:inertial_cylinder>
    </link>
@@ -74,8 +91,9 @@
    </gazebo>
    <!--RIGHT WHEEL LINK-->
+   <!-- <joint name="right_wheel_joint" type="continuous"> -->
    <joint name="right_wheel_joint" type="continuous">
       <parent link="base_link"/>
       <child link="right_wheel"/>
-      <origin xyz="0.0 -0.175 0.0" rpy="${pi/2} 0.0 0.0"/>
+      <origin xyz="0 ${-wheel_offset_y} ${-wheel_offset_z}" rpy="${pi/2} 0 0" />
       <axis xyz="0.0 0.0 -1"/>
    </joint>
@@ -83,5 +101,5 @@
       <visual>
          <geometry>
-            <cylinder radius="0.05" length="0.04"/>
+            <cylinder radius="${wheel_radius}" length="${wheel_thickness}"/>
          </geometry>
          <material name="blue"/>
@@ -89,8 +107,8 @@
       <collision>
          <geometry>
-            <cylinder radius="0.05" length="0.04"/>
+            <sphere radius="${wheel_radius}"/>
          </geometry>
       </collision>
-      <xacro:inertial_cylinder mass="0.1" length="0.04" radius="0.05">
+      <xacro:inertial_cylinder mass="${wheel_mass}" length="${wheel_thickness}" radius="${wheel_radius}">
          <origin xyz="0.0 0.0 0.0" rpy="0.0 0.0 0.0"/>
       </xacro:inertial_cylinder>
@@ -99,28 +117,55 @@
       <material>Gazebo/Blue</material>
    </gazebo>
-   <!-- CASTER WHEEL LINK -->
-   <joint name="caster_wheel_joint" type="fixed">
+   <!-- RIGHT CASTER WHEEL LINK -->
+   <joint name="right_caster_wheel_joint" type="fixed">
       <parent link="chassis"/>
-      <child link="caster_wheel"/>
-      <origin xyz="0.24 0.0 0.0"/>
+      <child link="right_caster_wheel"/>
+      <origin xyz="${caster_wheel_offset_x} ${-caster_wheel_offset_y} ${-caster_wheel_offset_z}"/>
    </joint>
-   <link name="caster_wheel">
+   <link name="right_caster_wheel">
       <visual>
          <geometry>
-            <sphere radius="0.05"/>
+            <sphere radius="${caster_wheel_radius}"/>
          </geometry>
-         <material name="black"/>
+         <material name="white"/>
       </visual>
       <collision>
          <geometry>
-            <sphere radius="0.05"/>
+            <sphere radius="${caster_wheel_radius}"/>
          </geometry>
       </collision>
-      <xacro:inertial_sphere mass="0.1" radius="0.05">
+      <xacro:inertial_sphere mass="${caster_wheel_mass}" radius="${caster_wheel_radius}">
          <origin xyz="0.0 0.0 0.0" rpy="0.0 0.0 0.0"/>
       </xacro:inertial_sphere>
    </link>
-   <gazebo reference="caster_wheel">
-      <material>Gazebo/Black</material>
+   <gazebo reference="right_caster_wheel">
+      <material>Gazebo/White</material>
+      <mu1 value="0.001"/>
+      <mu2 value="0.001"/>
+   </gazebo>
+   <!-- LEFT CASTER WHEEL LINK -->
+   <joint name="left_caster_wheel_joint" type="fixed">
+      <parent link="chassis"/>
+      <child link="left_caster_wheel"/>
+      <origin xyz="${caster_wheel_offset_x} ${caster_wheel_offset_y} ${-caster_wheel_offset_z}"/>
+   </joint>
+   <link name="left_caster_wheel">
+      <visual>
+         <geometry>
+            <sphere radius="${caster_wheel_radius}"/>
+         </geometry>
+         <material name="white"/>
+      </visual>
+      <collision>
+         <geometry>
+            <sphere radius="${caster_wheel_radius}"/>
+         </geometry>
+      </collision>
+      <xacro:inertial_sphere mass="${caster_wheel_mass}" radius="${caster_wheel_radius}">
+         <origin xyz="0.0 0.0 0.0" rpy="0.0 0.0 0.0"/>
+      </xacro:inertial_sphere>
+   </link>
+   <gazebo reference="left_caster_wheel">
+      <material>Gazebo/White</material>
       <mu1 value="0.001"/>
       <mu2 value="0.001"/>
