Commit message: add Simulating Sensors in Gazebo

File: description/lidar.xacro (robot description, xacro)
@@ -22,3 +22,31 @@
          </xacro:inertial_cylinder>
     </link>
+    <gazebo reference="laser_frame">
+        <material>Gazebo/Red</material>
+        <sensor name="laser" type="ray">
+            <pose> 0 0 0 0 0 0 </pose>
+            <visualize>true</visualize>
+            <update_rate>10</update_rate>
+            <ray>
+                <scan>
+                    <horizontal>
+                        <samples>360</samples>
+                        <min_angle>-3.14</min_angle>
+                        <max_angle>3.14</max_angle>
+                    </horizontal>
+                </scan>
+                <range>
+                    <min>0.3</min>
+                    <max>12</max>
+                </range>
+                <plugin name="laser_controller" filename="libgazebo_ros_ray_sensor.so">
+                    <ros>
+                        <argument>~/out:=scan</argument>
+                    </ros>
+                    <output_type>sensor_msgs/LaserScan</output_type>
+                    <frame_name>laser_frame</frame_name>
+                </plugin>
+            </ray>
+        </sensor>
+    </gazebo>
 </robot>

Commit message: Testing & Visualisation

File: description/lidar.xacro (robot description, xacro)
@@ -40,12 +40,12 @@
                     <max>12</max>
                 </range>
-                <plugin name="laser_controller" filename="libgazebo_ros_ray_sensor.so">
-                    <ros>
-                        <argument>~/out:=scan</argument>
-                    </ros>
-                    <output_type>sensor_msgs/LaserScan</output_type>
-                    <frame_name>laser_frame</frame_name>
-                </plugin>
             </ray>
+            <plugin name="laser_controller" filename="libgazebo_ros_ray_sensor.so">
+                <ros>
+                    <argument>~/out:=scan</argument>
+                </ros>
+                <output_type>sensor_msgs/LaserScan</output_type>
+                <frame_name>laser_frame</frame_name>
+            </plugin>
         </sensor>
     </gazebo>

File: description/robot_core.xacro (robot description, xacro)
@@ -73,56 +73,56 @@
       <material>Gazebo/Blue</material>
    </gazebo>
-      <!--RIGHT WHEEL LINK-->
-      <joint name="right_wheel_joint" type="continuous">
-         <parent link="base_link"/>
-         <child link="right_wheel"/>
-         <origin xyz="0.0 -0.175 0.0" rpy="${pi/2} 0.0 0.0"/>
-         <axis xyz="0.0 0.0 -1"/>
-      </joint>
-      <link name="right_wheel">
-         <visual>
-            <geometry>
-               <cylinder radius="0.05" length="0.04"/>
-            </geometry>
-            <material name="blue"/>
-         </visual>
-         <collision>
-            <geometry>
-               <cylinder radius="0.05" length="0.04"/>
-            </geometry>
-         </collision>
-         <xacro:inertial_cylinder mass="0.1" length="0.04" radius="0.05">
-            <origin xyz="0.0 0.0 0.0" rpy="0.0 0.0 0.0"/>
-         </xacro:inertial_cylinder>
-      </link>
-      <gazebo reference="right_wheel">
-         <material>Gazebo/Blue</material>
-      </gazebo>
-      <!-- CASTER WHEEL LINK -->
-      <joint name="caster_wheel_joint" type="fixed">
-         <parent link="chassis"/>
-         <child link="caster_wheel"/>
-         <origin xyz="0.24 0.0 0.0"/>
-      </joint>
-      <link name="caster_wheel">
-         <visual>
-            <geometry>
-               <sphere radius="0.05"/>
-            </geometry>
-            <material name="black"/>
-         </visual>
-         <collision>
-            <geometry>
-               <sphere radius="0.05"/>
-            </geometry>
-         </collision>
-         <xacro:inertial_sphere mass="0.1" radius="0.05">
-            <origin xyz="0.0 0.0 0.0" rpy="0.0 0.0 0.0"/>
-         </xacro:inertial_sphere>
-      </link>
-      <gazebo reference="caster_wheel">
-         <material>Gazebo/Black</material>
-         <mu1 value="0.001"/>
-         <mu2 value="0.001"/>
-      </gazebo>
+   <!--RIGHT WHEEL LINK-->
+   <joint name="right_wheel_joint" type="continuous">
+      <parent link="base_link"/>
+      <child link="right_wheel"/>
+      <origin xyz="0.0 -0.175 0.0" rpy="${pi/2} 0.0 0.0"/>
+      <axis xyz="0.0 0.0 -1"/>
+   </joint>
+   <link name="right_wheel">
+      <visual>
+         <geometry>
+            <cylinder radius="0.05" length="0.04"/>
+         </geometry>
+         <material name="blue"/>
+      </visual>
+      <collision>
+         <geometry>
+            <cylinder radius="0.05" length="0.04"/>
+         </geometry>
+      </collision>
+      <xacro:inertial_cylinder mass="0.1" length="0.04" radius="0.05">
+         <origin xyz="0.0 0.0 0.0" rpy="0.0 0.0 0.0"/>
+      </xacro:inertial_cylinder>
+   </link>
+   <gazebo reference="right_wheel">
+      <material>Gazebo/Blue</material>
+   </gazebo>
+   <!-- CASTER WHEEL LINK -->
+   <joint name="caster_wheel_joint" type="fixed">
+      <parent link="chassis"/>
+      <child link="caster_wheel"/>
+      <origin xyz="0.24 0.0 0.0"/>
+   </joint>
+   <link name="caster_wheel">
+      <visual>
+         <geometry>
+            <sphere radius="0.05"/>
+         </geometry>
+         <material name="black"/>
+      </visual>
+      <collision>
+         <geometry>
+            <sphere radius="0.05"/>
+         </geometry>
+      </collision>
+      <xacro:inertial_sphere mass="0.1" radius="0.05">
+         <origin xyz="0.0 0.0 0.0" rpy="0.0 0.0 0.0"/>
+      </xacro:inertial_sphere>
+   </link>
+   <gazebo reference="caster_wheel">
+      <material>Gazebo/Black</material>
+      <mu1 value="0.001"/>
+      <mu2 value="0.001"/>
+   </gazebo>
 </robot>

Commit message: try slam toolbox

File: description/lidar.xacro (robot description, xacro)
@@ -28,5 +28,6 @@
         <sensor name="laser" type="ray">
             <pose> 0 0 0 0 0 0 </pose>
-            <visualize>true</visualize>
+             <!-- <visualize>true</visualize> -->
+            <visualize>false</visualize>
             <update_rate>10</update_rate>
             <ray>

File: description/robot_core.xacro (robot description, xacro)
@@ -35,4 +35,12 @@
    <!-- BASE LINK -->
    <link name="base_link">
+   </link>
+   <!-- BASE_FOOTPRINT LINK -->
+   <joint name="base_footprint_joint" type="fixed">
+      <parent link="base_link"/>
+      <child link="base_footprint"/>
+      <origin xyz="0 0 0" rpy="0 0 0"/>
+   </joint>
+   <link name="base_footprint">
    </link>
    <!-- CHASSIS LINK -->
