Commit message: Created core URDF

File: description/robot_core.xacro (robot description, xacro)
@@ -41,4 +41,7 @@
       </xacro:inertial_box>
    </link>
+   <gazebo reference="chassis">
+      <material>Gazebo/White</material>
+   </gazebo>
    <!--LEFT WHEEL LINK-->
    <joint name="left_wheel_joint" type="continuous">
@@ -64,4 +67,7 @@
       </xacro:inertial_cylinder>
    </link>
+   <gazebo reference="left_wheel">
+      <material>Gazebo/Blue</material>
+   </gazebo>
       <!--RIGHT WHEEL LINK-->
       <joint name="right_wheel_joint" type="continuous">
@@ -87,4 +93,7 @@
          </xacro:inertial_cylinder>
       </link>
+      <gazebo reference="right_wheel">
+         <material>Gazebo/Blue</material>
+      </gazebo>
       <!-- CASTER WHEEL LINK -->
       <joint name="caster_wheel_joint" type="fixed">
@@ -109,3 +118,8 @@
          </xacro:inertial_sphere>
       </link>
+      <gazebo reference="caster_wheel">
+         <material>Gazebo/Black</material>
+         <mu1 value="0.001"/>
+         <mu2 value="0.001"/>
+      </gazebo>
 </robot>

Commit message: modify robot URDF

File: description/robot_core.xacro (robot description, xacro)
@@ -6,4 +6,5 @@
    <xacro:property name="chassis_width" value="0.154"/>
    <xacro:property name="chassis_height" value="0.128"/>
+   <xacro:property name="chassis_offset_z" value="0.07"/>
    <xacro:property name="chassis_mass" value="1.0"/>
    <xacro:property name="wheel_radius" value="0.040"/>
@@ -12,10 +13,11 @@
    <xacro:property name="wheel_offset_x" value="0.04"/>
    <xacro:property name="wheel_offset_y" value="0.107"/>
-   <xacro:property name="wheel_offset_z" value="0.0315"/>
+   <!-- <xacro:property name="wheel_offset_z" value="0.0315"/> -->
+   <xacro:property name="wheel_offset_z" value="0.04"/>
    <xacro:property name="caster_wheel_radius" value="0.0079"/>
    <xacro:property name="caster_wheel_mass" value="0.01"/>
    <xacro:property name="caster_wheel_offset_x" value="0.207"/>
    <xacro:property name="caster_wheel_offset_y" value="0.0485"/>
-   <xacro:property name="caster_wheel_offset_z" value="${wheel_offset_z + wheel_radius - caster_wheel_radius}"/>
+   <xacro:property name="caster_wheel_offset_z" value="${chassis_offset_z - caster_wheel_radius}"/>
    <material name="white">
       <color rgba="1 1 1 1"/>
@@ -48,5 +50,5 @@
       <parent link="base_link"/>
       <child link="chassis"/>
-      <origin xyz="${-wheel_offset_x} 0 0"/>
+      <origin xyz="${-wheel_offset_x} 0 ${chassis_offset_z}"/>
    </joint>
    <link name="chassis">
@@ -72,9 +74,9 @@
    </gazebo>
    <!--LEFT WHEEL LINK-->
-   <!-- <joint name="left_wheel_joint" type="continuous"> -->
+   <!-- <joint name="left_wheel_joint" type="fixed"> -->
    <joint name="left_wheel_joint" type="continuous">
       <parent link="base_link"/>
       <child link="left_wheel"/>
-      <origin xyz="0 ${wheel_offset_y} ${-wheel_offset_z}" rpy="-${pi/2} 0 0" />
+      <origin xyz="0 ${wheel_offset_y} ${wheel_offset_z}" rpy="-${pi/2} 0 0" />
       <axis xyz="0.0 0.0 1"/>
    </joint>
@@ -99,9 +101,9 @@
    </gazebo>
    <!--RIGHT WHEEL LINK-->
-   <!-- <joint name="right_wheel_joint" type="continuous"> -->
+   <!-- <joint name="right_wheel_joint" type="fixed"> -->
    <joint name="right_wheel_joint" type="continuous">
       <parent link="base_link"/>
       <child link="right_wheel"/>
-      <origin xyz="0 ${-wheel_offset_y} ${-wheel_offset_z}" rpy="${pi/2} 0 0" />
+      <origin xyz="0 ${-wheel_offset_y} ${wheel_offset_z}" rpy="${pi/2} 0 0" />
       <axis xyz="0.0 0.0 -1"/>
    </joint>
